Commit message: file renaming, configuration changes

File: hector_quadrotor_description/urdf/quadrotor_hokuyo_utm30lx.urdf.xacro (robot description, xacro)
@@ -6,14 +6,13 @@
     <!-- Instantiate quadrotor_base_macro once (has no parameters atm) -->
     <xacro:quadrotor_base_macro />
-    <!-- Hokuyo UTM-30LX mounted upside down below the quadrotor body -->
-    <xacro:include filename="$(find hector_sensors_description)/urdf/hokuyo_utm30lx.urdf.xacro" />
-    <xacro:hokuyo_utm30lx name="laser0" parent="base_link" ros_topic="scan" update_rate="40" ray_count="1081" min_angle="-135" max_angle="135">
-      <origin xyz="0.05 0.0 -0.097" rpy="${M_PI} 0 0"/>
-    </xacro:hokuyo_utm30lx>
     <!-- Forward facing camera -->
     <!-- Asus Xiton Live Pro -->
     <xacro:include filename="$(find hector_sensors_description)/urdf/asus_camera.urdf.xacro" />
     <xacro:asus_camera name="asus_camera" parent="base_link">
-      <origin xyz="-0.05 0.0 -0.08" rpy="0 ${M_PI/2} 0"/>
+      <origin xyz="0.06 0.0 -0.05" rpy="0 ${M_PI/9} 0"/>
     </xacro:asus_camera>
+    <xacro:include filename="$(find hector_sensors_description)/urdf/generic_camera.urdf.xacro" />
+    <xacro:generic_camera name="downward_cam" parent="base_link" ros_topic="downward_camera/image" cam_info_topic="downward_camera/camera_info" update_rate="20" res_x="640" res_y="480" image_format="L8" hfov="100">
+      <origin xyz="0.18 0.0 -0.012" rpy="0 ${M_PI/2} 0"/>
+    </xacro:generic_camera>
 </robot>

Commit message: find contours and 5 closest point added

File: hector_quadrotor_description/urdf/quadrotor_hokuyo_utm30lx.urdf.xacro (robot description, xacro)
@@ -14,5 +14,5 @@
     <xacro:include filename="$(find hector_sensors_description)/urdf/generic_camera.urdf.xacro" />
     <xacro:generic_camera name="downward_cam" parent="base_link" ros_topic="downward_camera/image" cam_info_topic="downward_camera/camera_info" update_rate="20" res_x="640" res_y="480" image_format="L8" hfov="100">
-      <origin xyz="0.18 0.0 -0.012" rpy="0 ${M_PI/2} 0"/>
+      <origin xyz="0.3 0.0 -0.012" rpy="0 ${M_PI/2} 0"/>
     </xacro:generic_camera>
 </robot>
