Commit message: configuration files' names changed, asus rotated to the side

File: hector_quadrotor_description/urdf/quadrotor_main.gazebo.xacro (robot description, xacro)
@@ -1,5 +1,5 @@
 <?xml version="1.0"?>
 <robot name="quadrotor" xmlns:xacro="http://www.ros.org/wiki/xacro">
-    <xacro:include filename="$(find hector_quadrotor_description)/urdf/quadrotor_hokuyo_utm30lx.urdf.xacro" />
+    <xacro:include filename="$(find hector_quadrotor_description)/urdf/quadrotor_main.urdf.xacro" />
     <xacro:include filename="$(find hector_quadrotor_gazebo)/urdf/quadrotor_plugins.gazebo.xacro" />
 </robot>

File: hector_quadrotor_description/urdf/quadrotor_main.urdf.xacro (robot description, xacro)
@@ -10,5 +10,5 @@
     <xacro:include filename="$(find hector_sensors_description)/urdf/asus_camera.urdf.xacro" />
     <xacro:asus_camera name="asus_camera" parent="base_link">
-      <origin xyz="0.06 0.0 -0.05" rpy="0 ${M_PI/9} 0"/>
+      <origin xyz="0.03 -0.08 -0.05" rpy="0 ${M_PI/9} ${-M_PI/2}"/>
     </xacro:asus_camera>
     <xacro:include filename="$(find hector_sensors_description)/urdf/generic_camera.urdf.xacro" />
