Commit message: mvp for data collection

File: hector_quadrotor_description/urdf/quadrotor_main.urdf.xacro (robot description, xacro)
@@ -10,5 +10,5 @@
     <xacro:include filename="$(find hector_sensors_description)/urdf/asus_camera.urdf.xacro" />
     <xacro:asus_camera name="asus_camera" parent="base_link">
-      <origin xyz="0.03 -0.08 -0.05" rpy="0 ${M_PI/9} ${-M_PI/2}"/>
+      <origin xyz="0.0 -0.08 -0.05" rpy="0 ${M_PI/9} ${-M_PI/2}"/>
     </xacro:asus_camera>
     <xacro:include filename="$(find hector_sensors_description)/urdf/generic_camera.urdf.xacro" />

Commit message: mvp

File: hector_quadrotor_description/urdf/quadrotor_main.urdf.xacro (robot description, xacro)
@@ -10,5 +10,5 @@
     <xacro:include filename="$(find hector_sensors_description)/urdf/asus_camera.urdf.xacro" />
     <xacro:asus_camera name="asus_camera" parent="base_link">
-      <origin xyz="0.0 -0.08 -0.05" rpy="0 ${M_PI/9} ${-M_PI/2}"/>
+      <origin xyz="0.0 -0.08 -0.05" rpy="0 ${M_PI/6} ${-M_PI/2}"/>
     </xacro:asus_camera>
     <xacro:include filename="$(find hector_sensors_description)/urdf/generic_camera.urdf.xacro" />

File: hector_sensors_description/urdf/asus_camera.urdf.xacro (robot description, xacro)
@@ -84,6 +84,6 @@
             </image>
             <clip>
-              <near>0.5</near>
-              <far>9</far>
+              <near>0.3</near>
+              <far>5</far>
             </clip>
           </camera>

Commit message: line offset added

File: hector_quadrotor_description/urdf/quadrotor_main.urdf.xacro (robot description, xacro)
@@ -10,5 +10,5 @@
     <xacro:include filename="$(find hector_sensors_description)/urdf/asus_camera.urdf.xacro" />
     <xacro:asus_camera name="asus_camera" parent="base_link">
-      <origin xyz="0.0 -0.08 -0.05" rpy="0 ${M_PI/6} ${-M_PI/2}"/>
+      <origin xyz="0.0 -0.08 -0.05" rpy="0 ${M_PI/4} ${-M_PI/2}"/>
     </xacro:asus_camera>
     <xacro:include filename="$(find hector_sensors_description)/urdf/generic_camera.urdf.xacro" />

Commit message: current state

File: hector_quadrotor_description/urdf/quadrotor_main.urdf.xacro (robot description, xacro)
@@ -10,5 +10,5 @@
     <xacro:include filename="$(find hector_sensors_description)/urdf/asus_camera.urdf.xacro" />
     <xacro:asus_camera name="asus_camera" parent="base_link">
-      <origin xyz="0.0 -0.08 -0.05" rpy="0 ${M_PI/4} ${-M_PI/2}"/>
+      <origin xyz="0.1 -0.08 -0.07" rpy="0 ${M_PI/4} ${-M_PI/3}"/>
     </xacro:asus_camera>
     <xacro:include filename="$(find hector_sensors_description)/urdf/generic_camera.urdf.xacro" />

File: hector_sensors_description/urdf/asus_camera.urdf.xacro (robot description, xacro)
@@ -85,5 +85,5 @@
             <clip>
               <near>0.3</near>
-              <far>5</far>
+              <far>9</far>
             </clip>
           </camera>
